Commit message: 我不知道为什么他还是不动这个车

File: src/cleanbot_course_project/urdf/robot_vacuum.xacro (robot description, xacro)
@@ -4,10 +4,10 @@
   <link name="base_link">
     <inertial>
-      <origin xyz="0 0 0.025" rpy="0 0 0" />
+      <origin xyz="0 0 0.055" rpy="0 0 0" />
       <mass value="6.0" />
       <inertia ixx="0.043" iyy="0.043" izz="0.078" ixy="0" iyz="0" ixz="0" />
     </inertial>
     <visual>
-      <origin xyz="0 0 0.025" rpy="0 0 0" />
+      <origin xyz="0 0 0.055" rpy="0 0 0" />
       <geometry>
         <cylinder radius="0.19" length="0.05" />
@@ -18,5 +18,5 @@
     </visual>
     <collision>
-      <origin xyz="0 0 0.025" rpy="0 0 0" />
+      <origin xyz="0 0 0.055" rpy="0 0 0" />
       <geometry>
         <cylinder radius="0.19" length="0.05" />
@@ -171,20 +171,20 @@
     <parent link="base_link" />
     <child link="caster_link" />
-    <origin xyz="-0.13 0 -0.005" rpy="0 0 0" />
+    <origin xyz="-0.13 0 0.02" rpy="0 0 0" />
   </joint>
   <joint name="lidar_joint" type="fixed">
     <parent link="base_link" />
     <child link="lidar_link" />
-    <origin xyz="0.0 0.0 0.05" rpy="0 0 0" />
+    <origin xyz="0.0 0.0 0.095" rpy="0 0 0" />
   </joint>
   <joint name="camera_joint" type="fixed">
     <parent link="base_link" />
     <child link="camera_link" />
-    <origin xyz="0.13 0.0 0.055" rpy="0 0 0" />
+    <origin xyz="0.13 0.0 0.085" rpy="0 0 0" />
   </joint>
   <joint name="rgbd_joint" type="fixed">
     <parent link="base_link" />
     <child link="rgbd_link" />
-    <origin xyz="0.12 0.0 0.045" rpy="0 0 0" />
+    <origin xyz="0.12 0.0 0.075" rpy="0 0 0" />
   </joint>
   <gazebo reference="base_link">
@@ -232,5 +232,7 @@
       <odometryFrame>odom</odometryFrame>
       <robotBaseFrame>base_link</robotBaseFrame>
-      <publishWheelTF>true</publishWheelTF>
+      <publishWheelTF>false</publishWheelTF>
+      <publishOdomTF>true</publishOdomTF>
+      <publishTf>true</publishTf>
       <publishOdom>true</publishOdom>
       <publishWheelJointState>true</publishWheelJointState>
