Commit message: 红绿灯

File: src/cleanbot_course_project/urdf/cleanbot_waffle_pi.urdf.xacro (robot description, xacro)
@@ -6,6 +6,16 @@
   <xacro:property name="body_color_name" value="$(arg body_color)" />
   <xacro:property name="body_rgba" value="0.12 0.12 0.12 1.0" />
+  <xacro:property name="wheel_rgba" value="0.12 0.12 0.12 1.0" />
   <xacro:if value="${body_color_name == 'red'}">
     <xacro:property name="body_rgba" value="0.85 0.12 0.12 1.0" />
+    <xacro:property name="wheel_rgba" value="0.85 0.12 0.12 1.0" />
+  </xacro:if>
+  <xacro:if value="${body_color_name == 'blue'}">
+    <xacro:property name="body_rgba" value="0.12 0.18 0.85 1.0" />
+    <xacro:property name="wheel_rgba" value="0.12 0.18 0.85 1.0" />
+  </xacro:if>
+  <xacro:if value="${body_color_name == 'green'}">
+    <xacro:property name="body_rgba" value="0.12 0.72 0.20 1.0" />
+    <xacro:property name="wheel_rgba" value="0.12 0.72 0.20 1.0" />
   </xacro:if>
   <link name="base_footprint"/>
@@ -51,5 +61,7 @@
         <mesh filename="package://turtlebot3_description/meshes/wheels/left_tire.stl" scale="0.001 0.001 0.001"/>
       </geometry>
-      <material name="dark"/>
+      <material name="wheel">
+        <color rgba="${wheel_rgba}"/>
+      </material>
     </visual>
     <collision>
@@ -79,5 +91,7 @@
         <mesh filename="package://turtlebot3_description/meshes/wheels/right_tire.stl" scale="0.001 0.001 0.001"/>
       </geometry>
-      <material name="dark"/>
+      <material name="wheel">
+        <color rgba="${wheel_rgba}"/>
+      </material>
     </visual>
     <collision>
@@ -152,5 +166,7 @@
         <mesh filename="package://turtlebot3_description/meshes/sensors/lds.stl" scale="0.001 0.001 0.001"/>
       </geometry>
-      <material name="dark"/>
+      <material name="sensor">
+        <color rgba="${wheel_rgba}"/>
+      </material>
     </visual>
     <collision>
@@ -193,3 +209,72 @@
   </joint>
   <link name="camera_rgb_optical_frame"/>
+  <xacro:if value="${body_color_name == 'blue'}">
+    <gazebo reference="base_link">
+      <material>Gazebo/Blue</material>
+    </gazebo>
+    <gazebo reference="wheel_left_link">
+      <material>Gazebo/Blue</material>
+    </gazebo>
+    <gazebo reference="wheel_right_link">
+      <material>Gazebo/Blue</material>
+    </gazebo>
+    <gazebo reference="base_scan">
+      <material>Gazebo/Blue</material>
+    </gazebo>
+  </xacro:if>
+  <xacro:if value="${body_color_name == 'green'}">
+    <gazebo reference="base_link">
+      <material>Gazebo/Green</material>
+    </gazebo>
+    <gazebo reference="wheel_left_link">
+      <material>Gazebo/Green</material>
+    </gazebo>
+    <gazebo reference="wheel_right_link">
+      <material>Gazebo/Green</material>
+    </gazebo>
+    <gazebo reference="base_scan">
+      <material>Gazebo/Green</material>
+    </gazebo>
+  </xacro:if>
+  <xacro:if value="${body_color_name == 'red'}">
+    <gazebo reference="base_link">
+      <material>Gazebo/Red</material>
+    </gazebo>
+    <gazebo reference="wheel_left_link">
+      <material>Gazebo/Red</material>
+    </gazebo>
+    <gazebo reference="wheel_right_link">
+      <material>Gazebo/Red</material>
+    </gazebo>
+    <gazebo reference="base_scan">
+      <material>Gazebo/Red</material>
+    </gazebo>
+  </xacro:if>
+  <gazebo reference="camera_link">
+    <sensor type="camera" name="cleanbot_rgb_camera">
+      <always_on>true</always_on>
+      <update_rate>30</update_rate>
+      <visualize>true</visualize>
+      <camera name="cleanbot_camera">
+        <horizontal_fov>1.047</horizontal_fov>
+        <image>
+          <width>640</width>
+          <height>480</height>
+          <format>R8G8B8</format>
+        </image>
+        <clip>
+          <near>0.05</near>
+          <far>8.0</far>
+        </clip>
+      </camera>
+      <plugin name="cleanbot_camera_controller" filename="libgazebo_ros_camera.so">
+        <alwaysOn>true</alwaysOn>
+        <updateRate>30.0</updateRate>
+        <cameraName>camera</cameraName>
+        <imageTopicName>rgb/image_raw</imageTopicName>
+        <cameraInfoTopicName>rgb/camera_info</cameraInfoTopicName>
+        <frameName>camera_rgb_optical_frame</frameName>
+      </plugin>
+    </sensor>
+  </gazebo>
 </robot>

Commit message: finial

File: src/cleanbot_course_project/urdf/cleanbot_waffle_pi.urdf.xacro (robot description, xacro)
@@ -2,7 +2,16 @@
 <robot name="turtlebot3_waffle_pi" xmlns:xacro="http://ros.org/wiki/xacro">
   <xacro:include filename="$(find turtlebot3_description)/urdf/common_properties.xacro"/>
-  <xacro:include filename="$(find turtlebot3_description)/urdf/turtlebot3_waffle_pi.gazebo.xacro"/>
+  <xacro:arg name="laser_visual" default="false" />
+  <xacro:arg name="imu_visual" default="false" />
   <xacro:arg name="body_color" default="dark" />
+  <xacro:arg name="enable_rgbd_camera" default="true" />
+  <xacro:arg name="frame_prefix" default="" />
   <xacro:property name="body_color_name" value="$(arg body_color)" />
+  <xacro:property name="frame_prefix_name" value="$(arg frame_prefix)" />
+  <xacro:property name="odom_frame_name" value="${frame_prefix_name + '/odom' if frame_prefix_name else 'odom'}" />
+  <xacro:property name="base_footprint_frame_name" value="${frame_prefix_name + '/base_footprint' if frame_prefix_name else 'base_footprint'}" />
+  <xacro:property name="base_scan_frame_name" value="${frame_prefix_name + '/base_scan' if frame_prefix_name else 'base_scan'}" />
+  <xacro:property name="imu_frame_name" value="${frame_prefix_name + '/imu_link' if frame_prefix_name else 'imu_link'}" />
+  <xacro:property name="camera_rgb_optical_frame_name" value="${frame_prefix_name + '/camera_rgb_optical_frame' if frame_prefix_name else 'camera_rgb_optical_frame'}" />
   <xacro:property name="body_rgba" value="0.12 0.12 0.12 1.0" />
   <xacro:property name="wheel_rgba" value="0.12 0.12 0.12 1.0" />
@@ -184,29 +193,57 @@
     </inertial>
   </link>
-  <joint name="camera_joint" type="fixed">
-    <origin xyz="0.073 -0.011 0.084" rpy="0 0 0"/>
-    <parent link="base_link"/>
-    <child link="camera_link"/>
-  </joint>
-  <link name="camera_link">
-    <collision>
-      <origin xyz="0.005 0.011 0.013" rpy="0 0 0"/>
-      <geometry>
-        <box size="0.015 0.030 0.027"/>
-      </geometry>
-    </collision>
-  </link>
-  <joint name="camera_rgb_joint" type="fixed">
-    <origin xyz="0.003 0.011 0.009" rpy="0 0 0"/>
-    <parent link="camera_link"/>
-    <child link="camera_rgb_frame"/>
-  </joint>
-  <link name="camera_rgb_frame"/>
-  <joint name="camera_rgb_optical_joint" type="fixed">
-    <origin xyz="0 0 0" rpy="-1.57 0 -1.57"/>
-    <parent link="camera_rgb_frame"/>
-    <child link="camera_rgb_optical_frame"/>
-  </joint>
-  <link name="camera_rgb_optical_frame"/>
+  <xacro:if value="$(arg enable_rgbd_camera)">
+    <joint name="camera_joint" type="fixed">
+      <origin xyz="0.073 -0.011 0.084" rpy="0 0 0"/>
+      <parent link="base_link"/>
+      <child link="camera_link"/>
+    </joint>
+    <link name="camera_link">
+      <inertial>
+        <origin xyz="0 0 0" rpy="0 0 0"/>
+        <mass value="0.08"/>
+        <inertia ixx="1.5e-05" ixy="0" ixz="0" iyy="1.5e-05" iyz="0" izz="1.5e-05"/>
+      </inertial>
+      <visual>
+        <origin xyz="0 0 0" rpy="0 0 0"/>
+        <geometry>
+          <box size="0.05 0.04 0.03"/>
+        </geometry>
+        <material name="camera">
+          <color rgba="0.82 0.82 0.82 1.0"/>
+        </material>
+      </visual>
+      <collision>
+        <origin xyz="0 0 0" rpy="0 0 0"/>
+        <geometry>
+          <box size="0.05 0.04 0.03"/>
+        </geometry>
+      </collision>
+    </link>
+    <joint name="camera_rgb_joint" type="fixed">
+      <origin xyz="0.003 0.011 0.009" rpy="0 0 0"/>
+      <parent link="camera_link"/>
+      <child link="camera_rgb_frame"/>
+    </joint>
+    <link name="camera_rgb_frame"/>
+    <joint name="camera_rgb_optical_joint" type="fixed">
+      <origin xyz="0 0 0" rpy="-1.57 0 -1.57"/>
+      <parent link="camera_rgb_frame"/>
+      <child link="camera_rgb_optical_frame"/>
+    </joint>
+    <link name="camera_rgb_optical_frame"/>
+    <joint name="camera_depth_joint" type="fixed">
+      <origin xyz="0.003 0.011 0.009" rpy="0 0 0"/>
+      <parent link="camera_link"/>
+      <child link="camera_depth_frame"/>
+    </joint>
+    <link name="camera_depth_frame"/>
+    <joint name="camera_depth_optical_joint" type="fixed">
+      <origin xyz="0 0 0" rpy="-1.57 0 -1.57"/>
+      <parent link="camera_depth_frame"/>
+      <child link="camera_depth_optical_frame"/>
+    </joint>
+    <link name="camera_depth_optical_frame"/>
+  </xacro:if>
   <xacro:if value="${body_color_name == 'blue'}">
     <gazebo reference="base_link">
@@ -251,28 +288,172 @@
     </gazebo>
   </xacro:if>
-  <gazebo reference="camera_link">
-    <sensor type="camera" name="cleanbot_rgb_camera">
+  <xacro:if value="$(arg enable_rgbd_camera)">
+    <gazebo reference="camera_rgb_frame">
+      <sensor type="depth" name="cleanbot_rgbd_camera">
+        <always_on>true</always_on>
+        <update_rate>30</update_rate>
+        <visualize>false</visualize>
+        <camera name="cleanbot_camera">
+          <horizontal_fov>1.3439</horizontal_fov>
+          <image>
+            <width>640</width>
+            <height>480</height>
+            <format>R8G8B8</format>
+          </image>
+          <depth_camera></depth_camera>
+          <clip>
+            <near>0.03</near>
+            <far>100</far>
+          </clip>
+        </camera>
+        <plugin name="cleanbot_rgbd_controller" filename="libgazebo_ros_openni_kinect.so">
+          <alwaysOn>true</alwaysOn>
+          <updateRate>30.0</updateRate>
+          <cameraName>camera</cameraName>
+          <frameName>${camera_rgb_optical_frame_name}</frameName>
+          <imageTopicName>rgb/image_raw</imageTopicName>
+          <cameraInfoTopicName>rgb/camera_info</cameraInfoTopicName>
+          <depthImageTopicName>depth/image_raw</depthImageTopicName>
+          <depthImageCameraInfoTopicName>depth/camera_info</depthImageCameraInfoTopicName>
+          <pointCloudTopicName>depth/points</pointCloudTopicName>
+          <pointCloudCutoff>0.4</pointCloudCutoff>
+          <hackBaseline>0.07</hackBaseline>
+          <CxPrime>0.0</CxPrime>
+          <Cx>0.0</Cx>
+          <Cy>0.0</Cy>
+          <focalLength>0</focalLength>
+        </plugin>
+      </sensor>
+    </gazebo>
+  </xacro:if>
+  <xacro:if value="${body_color_name == 'dark'}">
+    <gazebo reference="base_link">
+      <material>Gazebo/DarkGrey</material>
+    </gazebo>
+  </xacro:if>
+  <gazebo reference="wheel_left_link">
+    <mu1>0.1</mu1>
+    <mu2>0.1</mu2>
+    <kp>500000.0</kp>
+    <kd>10.0</kd>
+    <minDepth>0.001</minDepth>
+    <maxVel>0.1</maxVel>
+    <fdir1>1 0 0</fdir1>
+    <material>Gazebo/FlatBlack</material>
+  </gazebo>
+  <gazebo reference="wheel_right_link">
+    <mu1>0.1</mu1>
+    <mu2>0.1</mu2>
+    <kp>500000.0</kp>
+    <kd>10.0</kd>
+    <minDepth>0.001</minDepth>
+    <maxVel>0.1</maxVel>
+    <fdir1>1 0 0</fdir1>
+    <material>Gazebo/FlatBlack</material>
+  </gazebo>
+  <gazebo reference="caster_back_right_link">
+    <mu1>0.1</mu1>
+    <mu2>0.1</mu2>
+    <kp>1000000.0</kp>
+    <kd>100.0</kd>
+    <minDepth>0.001</minDepth>
+    <maxVel>1.0</maxVel>
+    <material>Gazebo/FlatBlack</material>
+  </gazebo>
+  <gazebo reference="caster_back_left_link">
+    <mu1>0.1</mu1>
+    <mu2>0.1</mu2>
+    <kp>1000000.0</kp>
+    <kd>100.0</kd>
+    <minDepth>0.001</minDepth>
+    <maxVel>1.0</maxVel>
+    <material>Gazebo/FlatBlack</material>
+  </gazebo>
+  <gazebo reference="imu_link">
+    <sensor type="imu" name="imu">
       <always_on>true</always_on>
-      <update_rate>30</update_rate>
-      <visualize>true</visualize>
-      <camera name="cleanbot_camera">
-        <horizontal_fov>1.047</horizontal_fov>
-        <image>
-          <width>640</width>
-          <height>480</height>
-          <format>R8G8B8</format>
-        </image>
-        <clip>
-          <near>0.05</near>
-          <far>8.0</far>
-        </clip>
-      </camera>
-      <plugin name="cleanbot_camera_controller" filename="libgazebo_ros_camera.so">
-        <alwaysOn>true</alwaysOn>
-        <updateRate>30.0</updateRate>
-        <cameraName>camera</cameraName>
-        <imageTopicName>rgb/image_raw</imageTopicName>
-        <cameraInfoTopicName>rgb/camera_info</cameraInfoTopicName>
-        <frameName>camera_rgb_optical_frame</frameName>
+      <visualize>$(arg imu_visual)</visualize>
+    </sensor>
+    <material>Gazebo/Grey</material>
+  </gazebo>
+  <gazebo>
+    <plugin name="turtlebot3_waffle_pi_controller" filename="libgazebo_ros_diff_drive.so">
+      <commandTopic>cmd_vel</commandTopic>
+      <odometryTopic>odom</odometryTopic>
+      <odometryFrame>${odom_frame_name}</odometryFrame>
+      <odometrySource>world</odometrySource>
+      <publishOdomTF>true</publishOdomTF>
+      <robotBaseFrame>${base_footprint_frame_name}</robotBaseFrame>
+      <publishWheelTF>false</publishWheelTF>
+      <publishTf>true</publishTf>
+      <publishWheelJointState>true</publishWheelJointState>
+      <legacyMode>false</legacyMode>
+      <updateRate>30</updateRate>
+      <leftJoint>wheel_left_joint</leftJoint>
+      <rightJoint>wheel_right_joint</rightJoint>
+      <wheelSeparation>0.287</wheelSeparation>
+      <wheelDiameter>0.066</wheelDiameter>
+      <wheelAcceleration>1</wheelAcceleration>
+      <wheelTorque>10</wheelTorque>
+      <rosDebugLevel>na</rosDebugLevel>
+    </plugin>
+  </gazebo>
+  <gazebo>
+    <plugin name="imu_plugin" filename="libgazebo_ros_imu.so">
+      <alwaysOn>true</alwaysOn>
+      <bodyName>imu_link</bodyName>
+      <frameName>${imu_frame_name}</frameName>
+      <topicName>imu</topicName>
+      <serviceName>imu_service</serviceName>
+      <gaussianNoise>0.0</gaussianNoise>
+      <updateRate>0</updateRate>
+      <imu>
+        <noise>
+          <type>gaussian</type>
+          <rate>
+            <mean>0.0</mean>
+            <stddev>2e-4</stddev>
+            <bias_mean>0.0000075</bias_mean>
+            <bias_stddev>0.0000008</bias_stddev>
+          </rate>
+          <accel>
+            <mean>0.0</mean>
+            <stddev>1.7e-2</stddev>
+            <bias_mean>0.1</bias_mean>
+            <bias_stddev>0.001</bias_stddev>
+          </accel>
+        </noise>
+      </imu>
+    </plugin>
+  </gazebo>
+  <gazebo reference="base_scan">
+    <material>Gazebo/FlatBlack</material>
+    <sensor type="ray" name="lds_lfcd_sensor">
+      <pose>0 0 0 0 0 0</pose>
+      <visualize>$(arg laser_visual)</visualize>
+      <update_rate>5</update_rate>
+      <ray>
+        <scan>
+          <horizontal>
+            <samples>360</samples>
+            <resolution>1</resolution>
+            <min_angle>0.0</min_angle>
+            <max_angle>6.28319</max_angle>
+          </horizontal>
+        </scan>
+        <range>
+          <min>0.120</min>
+          <max>3.5</max>
+          <resolution>0.015</resolution>
+        </range>
+        <noise>
+          <type>gaussian</type>
+          <mean>0.0</mean>
+          <stddev>0.01</stddev>
+        </noise>
+      </ray>
+      <plugin name="gazebo_ros_lds_lfcd_controller" filename="libgazebo_ros_laser.so">
+        <topicName>scan</topicName>
+        <frameName>${base_scan_frame_name}</frameName>
       </plugin>
     </sensor>
